Commit message: creat a caster_wheel

File: robot_description/urdf/first_robot.urdf (robot description, URDF)
Before this commit: robot first_bot, 4 links, 3 joints
Links:
- added link caster_wheel, mass 2; collision sphere radius=0.05; visual sphere radius=0.05
Joints:
- added joint base_to_caster_wheel: type fixed, parent base_link, child caster_wheel, origin xyz=-0.225 0 -0.15

Commit message: try to creat lidar but failed

File: robot_description/urdf/first_robot.urdf (robot description, URDF)
Before this commit: robot first_bot, 5 links, 4 joints
Joints:
- joint base_to_lidar: origin xyz=0.3 0 0.13 -> xyz=0.2 0 0.15
